File: hw/pcb/controller.sch (EAGLE design)
At the start: 26 parts, among them IC1 MCP23017SS, Q1 MOSFET-NCH, U2 TMP102, U3 MCP6004, U4 MCP2510SO

Commit message: working aux control over mqtt; working multi-input and inversion
Parts:
- added D2: MMBZ, curtek:MMBZ_SOT23
- added IC2: 4001D, 40xx:4001D
- added R13: 10k, rcl:R-EU_R0603
- added R14, R15: 56k, rcl:R-EU_R0603
- added U$1: RESISTOR_INTERNAL_PULLUP, curtek:RESISTOR_INTERNAL_PULLUP
- R10: value 10k -> 100k
Connections:
- new net INPUT_1: R13.2, X5.1
- new net INPUT_2: X5.2
- new net INPUT_3: X5.3
- new net INPUT_4: X5.4
- new net INPUT_5: X5.5
- new net INPUT_6: X5.6
- new net INPUT_7: X5.7
- new net INPUT_8: X5.8
- new net N$13: IC2A.O, IC2B.I0
- new net N$15: IC2A.I0, R14.1
- new net N$16: IC2B.I1, R15.1
- new net N$17: IC2A.I1, IC2B.O
- new net N$21: X5.9
- new net N$22: X5.10
- new net N$23: X5.11
- new net N$24: X5.12
- new net N$9: D2.CATHODE_1
- net 3.3V: now also U$1.P$2
- net GND: now also D2.ANODE, R14.2, R15.2
- net INPUT_ACCESSORY: now also D2.CATHODE_2, R13.1
- net MCP_GPA0: now also U$1.P$1
Other:
- note added: "must be a rail-to-rail op-amp or else consider how close to the rails we can get -- otherwise we lose precious resolution"
- note added: "need power on reset circuit to force a particular state"
